Commit message: snart færdig med IMU demo

File: src/forklift_description/urdf/forklift_description.urdf (robot description, URDF)
Before this commit: robot forklift, 2 links, 1 joints
Links:
- link imu_link: geometry visual mesh filename=package://forklift_description/meshes/forklift_opt4.dae scale=0.001 0.001 0.001
Joints:
- joint world_to_imu: origin xyz=0 0 -0.5 rpy=0 0 0 -> xyz=0 0 0 rpy=0 0 0

Commit message: fjernet store dae filer

File: src/forklift_description/urdf/forklift_description.urdf (robot description, URDF)
Before this commit: robot forklift, 2 links, 1 joints
Links:
- link imu_link: geometry visual mesh filename=package://forklift_description/meshes/forklift.dae scale=0.001 0.001 0.001

Commit message: kæmpe rfid forbedringer

File: src/forklift_description/urdf/forklift_description.urdf (robot description, URDF)
Before this commit: robot forklift, 2 links, 1 joints
Links:
- removed link imu_link
- added link imu1_link
- added link imu2_link
- added link model_link; visual mesh filename=package://forklift_description/meshes/forklift.dae scale=0.001 0.001 0.001
Joints:
- removed joint world_to_imu
- added joint model_to_imu1: type fixed, parent model_link, child imu1_link, origin xyz=0 0 0 rpy=0 0 0
- added joint model_to_imu2: type fixed, parent model_link, child imu2_link, origin xyz=0.5 0 0 rpy=0 0 0
- added joint world_to_model: type fixed, parent world, child model_link, origin xyz=0 0 0 rpy=0 0 0
